File: PCB/e-ink_macropad/e-ink_macropad.kicad_pcb (KiCad board)
At the start: 2 copper layers, 77 parts, among them Q1 Si1308EDL, Q2 Si1308EDL, Q3 Si1308EDL, Q4 Si1308EDL, SW1 SW_Omron_B3FS, SW2 SW_Omron_B3FS, SW3 SW_Omron_B3FS, SW4 SW_Omron_B3FS, SW5 RotaryEncoder_Switch, U1 E-INK, U2 E-INK, U3 E-INK, U4 E-INK

Commit message: Finalised the PCB layout
Parts:
- SW1, SW2, SW3, SW4: value SW_Omron_B3FS -> SW_Cherry
- U5: footprint Library:MODULE_ESP32-C3_SUPERMINI_TH -> Library:MODULE_ESP32-C3_SUPERMINI
- moved D7 233.3 mm to (50.2, 138.5), turned to 0 degrees
- moved C31 229.9 mm to (48.6, 136.5)
- moved D9 226.9 mm to (55.5, 138.5), turned to 0 degrees
- moved C29 225.6 mm to (58.2, 143.0)
- moved R5 224.8 mm to (48.4, 146.0)
- moved C24 224.3 mm to (48.4, 119.5)
- moved Q3 224.2 mm to (52.0, 144.6), turned to 0 degrees
- moved C30 222.9 mm to (57.2, 136.5)
- moved R6 222.7 mm to (48.4, 143.5)
- moved D3 222.7 mm to (50.1, 121.5), turned to 0 degrees
- moved D8 222.5 mm to (60.8, 138.5), turned to 0 degrees
- moved L3 221.6 mm to (56.5, 144.8)
- moved D2 216.9 mm to (55.5, 121.5), turned to 0 degrees
- moved C32 216.7 mm to (62.4, 136.5)
- moved R2 212.4 mm to (49.4, 126.5)
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Connections:
- U1 pad MP: (no net) -> GND
- U2 pad MP: (no net) -> GND
- U3 pad MP: (no net) -> GND
- U4 pad MP: (no net) -> GND
Routing:
- net +3V3: track 0.00 -> 333.0 mm, vias 0 -> 6
- net /SPI_SCK: track 0.00 -> 219.5 mm, vias 0 -> 4
- net /EINK_DC: track 0.00 -> 206.0 mm, vias 0 -> 4
- net /EINK_RES: track 0.00 -> 205.9 mm, vias 0 -> 4
- net /EINK_BUSY: track 0.00 -> 193.8 mm, vias 0 -> 6
- net /SPI_MOSI: track 0.00 -> 153.0 mm, vias 0 -> 4
- net /BTN3: track 0.00 -> 147.5 mm
- net /BTN2: track 0.00 -> 125.5 mm
- net /DT: track 0.00 -> 92.2 mm
- net /SW: track 0.00 -> 91.9 mm
- net /CLK: track 0.00 -> 74.5 mm
- net /BTN4: track 0.00 -> 70.1 mm
- net /C/S_3: track 0.00 -> 66.3 mm
- net /C/S_4: track 0.00 -> 54.3 mm
- net /C/S_2: track 0.00 -> 45.6 mm
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- added copper zone on B.Cu, net GND
Other:
- board outline added: 87 x 66 mm
