File: PCB/e-ink_macropad/e-ink_macropad.kicad_sch (KiCad schematic)
At the start: 77 parts, among them Q1 Si1308EDL, Q2 Si1308EDL, Q3 Si1308EDL, Q4 Si1308EDL, SW1 SW_Omron_B3FS, SW2 SW_Omron_B3FS, SW3 SW_Omron_B3FS, SW4 SW_Omron_B3FS, SW5 RotaryEncoder_Switch, U1 E-INK, U2 E-INK, U3 E-INK, U4 E-INK

Commit message: Finalised the PCB layout
Parts:
- U5: footprint Library:MODULE_ESP32-C3_SUPERMINI_TH -> Library:MODULE_ESP32-C3_SUPERMINI
Changed lines of the file:
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@@
 			)
 		)
-		(property "Footprint" "Library:MODULE_ESP32-C3_SUPERMINI_TH"
+		(property "Footprint" "Library:MODULE_ESP32-C3_SUPERMINI"
 			(at 144.78 40.64 0)
 			(hide yes)
